Commit message: Working joint position and velocity control; need to tune on panda

File: examples/98-nullspace/ppbot.urdf (robot description, URDF)
Before this commit: robot RRRBot, 4 links, 3 joints
Links:
- removed link link3
- link link0: mass 1 -> 0.001; geometry 
- link link1: mass 1 -> 0.001; geometry 
- link link2: geometry visual cylinder length=0.04 radius=0.1
Joints:
- removed joint j3
- joint j0: axis 0 0 1 -> 1 0 0; type revolute -> prismatic
- joint j1: axis 0 0 1 -> 0 1 0; origin xyz=0.5 0 0 rpy=0 0 0 -> xyz=0 0 0 rpy=0 0 0; type revolute -> prismatic
